File: Hardware/Rev1/AT_HUB_RECHARGED/AT_HUB_RECHARGED.kicad_pcb (KiCad board)
At the start: 2 copper layers, 100 x 55 mm, 97 parts, among them J1 ESP Current SNS, J10 IN3, J11 IN4, J12 IN5, J13 Pack Thermister, J14 Through Hole, J15 EXT Charge Port, J16 USB_C_Receptacle_PowerOnly_6P, J2 JST, J3 OUT1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

Commit message: Done the design will verify
Routing:
- net +3V3: track 66.6 -> 86.5 mm
- net GND: track 113.3 -> 121.4 mm, vias 101 -> 210
