File: Hardware/Rev2/AT_HUB_RECHARGED/AT_HUB_RECHARGED.kicad_pcb (KiCad board)
At the start: 2 copper layers, 100 x 55 mm, 93 parts, among them J1 ESP Current SNS, J10 IN3, J11 IN4, J12 IN5, J13 Pack Thermister, J14 Through Hole, J15 EXT Charge Port, J16 USB_C_Receptacle_PowerOnly_6P, J2 JST, J3 OUT1, J4 OUT2, J5 OUT3, J6 OUT4, J7 OUT5, J8 IN1, J9 IN2, SW1 SW_Push, SW10 SW_Push, SW11 SW_SPDT, SW2 SW_Push, SW3 SW_Push, SW4 SW_Push, SW5 SW_Push, SW6 SW_Push, SW7 SW_Push, SW8 SW_Push, SW9 SW_Push, U1 ESP32-PICO-DEVKITM-2, U2 TLP241A(TP1,F, U3 TLP241A(TP1,F, U4 TLP241A(TP1,F, U5 TLP241A(TP1,F, U6 TLP241A(TP1,F, U7 BQ21040DBV, U8 TLV61070ADBV, U9 BQ27427YZFR

Commit message: Added new protections and load sharing for lipo, also changed inductor to be autoplaced
Parts:
- removed D8: CDBW140-G, Diode_SMD:D_SOD-123
- removed F1: 500mA, Fuse:Fuse_1206_3216Metric
- removed J1: ESP Current SNS, Connector_PinHeader_2.54mm:PinHeader_1x02_P2.54mm_Vertical
- added D9: 1N5819HW-7-F, Diode_SMD:D_SOD-123, F.Cu at (174.6, 93.2)
- added JP3: SKIP PMOS 2, Jumper:SolderJumper-2_P1.3mm_Open_RoundedPad1.0x1.5mm, B.Cu at (180.4, 110.7)
- added Q1: NTR1P02T1G, Package_TO_SOT_SMD:SOT-23, F.Cu at (182.2, 110.2)
- added Q2: NTR1P02T1G, Package_TO_SOT_SMD:SOT-23, F.Cu at (178.8, 110.2)
- added R29: 0R, Resistor_SMD:R_0805_2012Metric, F.Cu at (185.7, 109.2)
- added R30: 100k, Resistor_SMD:R_0805_2012Metric, F.Cu at (186.3, 92.5)
- C3: footprint Capacitor_SMD:C_1210_3225Metric -> Capacitor_SMD:C_1206_3216Metric
- C7, D11, D12, D13, D14, D15, R1, R11, R12, R13, R14, R15, R2, R20, R21, R22, R23, R24, R25, R26, R3, R4, R5: moved to F.Cu
- L1: footprint Inductor_SMD:L_Taiyo-Yuden_NR-60xx -> AT_HUB_R2:Ceaiya SMD,6x6mm CR6028-2R2N
- R27, R7: value 600R -> 1k; moved to F.Cu
- moved R15 39.0 mm to (138.3, 105.8)
- moved R20 11.7 mm to (181.3, 96.9)
- moved R25 9.05 mm to (100.0, 107.5), turned to -90 degrees
- moved D13 8.88 mm to (187.2, 83.2), turned to 0 degrees
- moved R26 8.32 mm to (102.0, 107.5), turned to 90 degrees
- moved C7 7.97 mm to (191.5, 91.2)
- moved L1 5.13 mm to (168.1, 98.6)
- moved R9 3.94 mm to (172.6, 111.8), turned to 180 degrees
- moved R3 3.64 mm to (153.4, 114.4)
- moved R1 3.62 mm to (117.5, 114.5)
- moved R2 3.62 mm to (135.5, 114.5)
- moved R5 3.61 mm to (189.6, 114.5)
- moved R4 3.56 mm to (171.4, 114.3)
- moved C4 3.50 mm to (175.4, 110.5)
- moved R22 2.80 mm to (152.1, 105.5)
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Connections:
- C4 pad 1: /Battery Management/Load/CHRG+ -> /Battery Management/SYS_LOAD
- J14 pad 2: Net-(J14-Pin_2) -> /Battery Management/Pack+
- J2 pad 1: Net-(J14-Pin_2) -> /Battery Management/Pack+
- L1 pad 1: /Battery Management/Load/CHRG+ -> /Battery Management/SYS_LOAD
- SW11 pad 3: /Battery Management/Load/CHRG+ -> /Battery Management/SYS_LOAD
- U1 pad 20: Net-(J1-Pin_2) -> unconnected-(U1-SENSOR_VP-Pad20)
- U1 pad 21: Net-(J1-Pin_1) -> unconnected-(U1-SENSOR_VM-Pad21)
- U8 pad 6: /Battery Management/Load/CHRG+ -> /Battery Management/SYS_LOAD
Routing:
- net /Battery Management/SYS_LOAD: track 0.00 -> 57.2 mm, vias 0 -> 4
- net Net-(D5-A): track 3.10 -> 45.7 mm
- net /PILOT_LED5: track 45.4 -> 4.21 mm, vias 2 -> 0
- net /Battery Management/Load/CHRG+: track 74.1 -> 107.7 mm, vias 2 -> 4
- net GND: track 21.8 -> 51.1 mm, vias 224 -> 189
- net VBUS: track 117.2 -> 142.3 mm, vias 0 -> 4
- net /Battery Management/Pack+: track 25.9 -> 45.3 mm, vias 2 -> 4
- net Net-(J14-Pin_2): track 14.9 -> 0.00 mm, vias 2 -> 0
- net unconnected-(U1-SENSOR_VP-Pad20): track 0.00 -> 14.5 mm
- net Net-(J1-Pin_2): track 14.5 -> 0.00 mm
- net unconnected-(U1-SENSOR_VM-Pad21): track 0.00 -> 14.5 mm
- net Net-(J1-Pin_1): track 14.5 -> 0.00 mm
- net Net-(U1-IO12): track 55.8 -> 68.4 mm, vias 1 -> 2
- net Net-(Q1-G): track 0.00 -> 7.29 mm
- net /RELAY3: track 55.7 -> 62.1 mm, vias 1 -> 2
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- added copper zone on F.Cu, net /Battery Management/SYS_LOAD

Commit message: Done the design will verify
Parts:
- removed C6: 2u2, Capacitor_SMD:C_0805_2012Metric
- removed C7: 1u, Capacitor_SMD:C_0805_2012Metric
- removed U9: BQ27427YZFR, AT_HUB_R2:IC_BQ27427YZFR
- added C8: 1u, Capacitor_SMD:C_0805_2012Metric, F.Cu at (192.9, 103.0)
- added C9: 2u2, Capacitor_SMD:C_0805_2012Metric, F.Cu at (185.3, 106.5)
- added R31: 10k, Resistor_SMD:R_0402_1005Metric, F.Cu at (138.8, 85.6)
- added R32: 10k, Resistor_SMD:R_0402_1005Metric, F.Cu at (149.1, 94.8)
- added R33: 10k, Resistor_SMD:R_0402_1005Metric, F.Cu at (116.0, 111.4)
- added R34: 10k, Resistor_SMD:R_0402_1005Metric, F.Cu at (135.9, 95.2)
- added R35: 10k, Resistor_SMD:R_0402_1005Metric, F.Cu at (134.2, 94.0)
- added R36: R01, Resistor_SMD:R_0805_2012Metric, F.Cu at (190.9, 103.0)
- added U10: BQ27441DRZR-G1A, Package_SON:Texas_S-PDSO-N12, F.Cu at (187.0, 102.8)
- L1: value 4u7 -> 2u2
- moved R17 76.9 mm to (112.4, 94.5)
- moved R16 72.9 mm to (114.4, 94.5)
- moved JP2 1.25 mm to (185.9, 98.0)
- moved R18 1.23 mm to (191.2, 106.5)
- moved R19 1.19 mm to (193.2, 106.5)
- moved R28 1.19 mm to (193.2, 106.5)
Connections:
- net /Battery Management/Load/CHRG+ renamed /Battery Management/Bat+
- U1 pad 15: /RELAY2 -> /BTN5
- U1 pad 22: /BTN5 -> /RELAY2
Routing:
- net +3V3: track 74.5 -> 170.7 mm, vias 2 -> 9
- net SDA: track 128.6 -> 90.2 mm, vias 3 -> 2
- net SCL: track 127.3 -> 89.3 mm, vias 3 -> 2
- net /BTN5: track 36.1 -> 63.8 mm, vias 0 -> 3
- net /Battery Management/VDD_GAUGE: track 15.3 -> 0.00 mm, vias 3 -> 0
- net unconnected-(U1-SENSOR_VP-Pad20): track 14.5 -> 0.00 mm
- net unconnected-(U1-SENSOR_VM-Pad21): track 14.5 -> 0.00 mm
- net /Battery Management/Bat+: track 107.7 -> 94.8 mm
- net /GAUGE_GPOUT: track 138.7 -> 129.6 mm
- net GND: track 51.1 -> 44.1 mm, vias 189 -> 231
- net /BTN4: track 37.8 -> 44.5 mm
- net VBUS: track 142.3 -> 147.1 mm, vias 4 -> 2
- net /BTN2: track 39.6 -> 44.4 mm, vias 1 -> 2
- net Net-(U10-V_{DD}): track 0.00 -> 3.96 mm
- net /BTN3: track 21.7 -> 25.5 mm, vias 0 -> 1
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- added copper zone on In1.Cu, net GND
- added copper zone on In2.Cu, net GND
- removed copper zone on F.Cu, net /Battery Management/Bat+
- removed copper zone on F.Cu, net /Battery Management/Pack+
Other:
- copper layers 2 -> 4

Commit message: Added Rev 3
Parts:
- removed R28: 10k, Resistor_SMD:R_0805_2012Metric
- C2: footprint Capacitor_SMD:C_Elec_6.3x7.7 -> Capacitor_Tantalum_SMD:CP_EIA-3216-18_Kemet-A
- R8: moved to F.Cu
- moved C2 1.40 mm to (99.2, 87.6)
- turned C8 to 90 degrees
Connections:
- C8 pad 1: /Battery Management/Pack+ -> /Battery Management/Bat+
- C9 pad 1: Net-(U10-V_{DD}) -> /Battery Management/VDD_GAUGE
- U10 pad 5: Net-(U10-V_{DD}) -> /Battery Management/VDD_GAUGE
Routing:
- net Net-(U10-V_{DD}): track 3.96 -> 0.00 mm
- net /Battery Management/VDD_GAUGE: track 0.00 -> 3.96 mm
- net /Battery Management/TS: track 13.9 -> 16.7 mm
- net /Battery Management/Bat+: track 94.8 -> 96.8 mm
- net Net-(U8-V_{FB}): track 1.97 -> 3.97 mm
- net /Battery Management/Pack+: track 45.5 -> 43.5 mm
- net VBUS: track 147.1 -> 148.6 mm
- net /BTN4: track 44.5 -> 43.1 mm
- net GND: track 44.1 -> 44.2 mm, vias 231 -> 230
