File: Hardware/Rev3/AT_HUB_RECHARGED/AT_HUB_RECHARGED.kicad_pcb (KiCad board)
At the start: 4 copper layers, 100 x 55 mm, 99 parts, among them J10 IN3, J11 IN4, J12 IN5, J13 Pack Thermister, J14 Through Hole, J15 EXT Charge Port, J16 USB_C_Receptacle_PowerOnly_6P, J2 JST, J3 OUT1, J4 OUT2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

Commit message: Final working
Parts:
- added R28: 10k, Resistor_SMD:R_0805_2012Metric, F.Cu at (113.7, 104.1)
Routing:
- net +3V3: track 170.7 -> 174.8 mm
- net /BACKUP_BTN1: track 10.2 -> 12.2 mm
